Commit message: modify: lidar1 pitch modified to 0deg

File: base_ws/src/vehicle/urdf/ioniq5.urdf.xacro (robot description, xacro)
@@ -5,8 +5,7 @@
       x forward, y left, z up.
       the baked mesh origin is the rear axle ground projection.
-    Runtime placement below assumes MORAI base_link is close to the rear axle
-    wheel center. The mesh is shifted down by the tire radius plus a small
-    LiDAR self-return alignment correction measured against MORAI ego-body
-    points around the hood and roof.
+    MORAI sensor extrinsics in configs/sensors/Sensor_1.json use the same
+    rear-axle ground base frame, so the visual/collision mesh must not be
+    shifted by wheel radius here.
     Visual mesh bbox:
       x [-0.790, 3.845]
@@ -20,7 +19,5 @@
   <xacro:property name="vehicle_center_x" value="1.5275"/>
   <xacro:property name="vehicle_center_z" value="0.800"/>
-  <xacro:property name="tire_radius" value="0.3705"/>
-  <xacro:property name="morai_body_lidar_z_correction" value="-0.0395"/>
-  <xacro:property name="visual_z_offset" value="${-tire_radius + morai_body_lidar_z_correction}"/>
+  <xacro:property name="visual_z_offset" value="0.0"/>
   <link name="base_link">
     <visual name="ioniq5_visual">

Commit message: add: GPS, IMU added

File: base_ws/src/vehicle/urdf/ioniq5.urdf.xacro (robot description, xacro)
@@ -2,14 +2,18 @@
 <robot name="ioniq5" xmlns:xacro="http://www.ros.org/wiki/xacro">
   <!--
-    Mesh coordinates are baked for ROS:
+    Mesh coordinates are baked for ROS with a rear-axle ground-projection origin:
       x forward, y left, z up.
-      the baked mesh origin is the rear axle ground projection.
-    MORAI sensor extrinsics in configs/sensors/Sensor_1.json use the same
-    rear-axle ground base frame, so the visual/collision mesh must not be
-    shifted by wheel radius here.
-    Visual mesh bbox:
+      the baked mesh origin is directly below the rear axle center.
+    Runtime base_link is the rear axle center, not the ground projection.
+    MORAI sensor extrinsics in configs/sensors/Sensor_1.json use that same
+    rear axle center frame. The visual/collision mesh is shifted downward by
+    the wheel radius so RViz shows the vehicle around the axle-centered
+    base_link correctly.
+    Baked visual mesh bbox before URDF origin offset:
       x [-0.790, 3.845]
       y [-1.067, 1.067]
       z [0.000, 1.600]
+    Runtime visual bbox after offset:
+      z [-0.3705, 1.2295]
   -->
   <xacro:property name="vehicle_length" value="4.635"/>
@@ -17,7 +21,9 @@
   <xacro:property name="vehicle_mirror_width" value="2.134"/>
   <xacro:property name="vehicle_height" value="1.600"/>
+  <xacro:property name="tire_outer_diameter" value="0.741"/>
+  <xacro:property name="wheel_radius" value="${tire_outer_diameter / 2.0}"/>
   <xacro:property name="vehicle_center_x" value="1.5275"/>
   <xacro:property name="vehicle_center_z" value="0.800"/>
-  <xacro:property name="visual_z_offset" value="0.0"/>
+  <xacro:property name="visual_z_offset" value="${-wheel_radius}"/>
   <link name="base_link">
     <visual name="ioniq5_visual">

Commit message: add: static tf between morai map <-> lanelet map (map)

File: base_ws/src/vehicle/urdf/ioniq5.urdf.xacro (robot description, xacro)
@@ -10,9 +10,18 @@
     the wheel radius so RViz shows the vehicle around the axle-centered
     base_link correctly.
+    MORAI's ego self-return in /sensor/lidar_concat does not expose the full
+    mesh silhouette uniformly. The visible front/roof bands measured against
+    the baked mesh first suggested about -0.10 m in x:
+      z 0.45..0.65 m: cloud front 3.634 m, mesh front 3.727 m
+      z 1.05..1.25 m: cloud front 1.841 m, mesh front 1.948 m
+    A live RViz visual check still showed the model behind the cloud, so the
+    displayed model was moved 0.05 m forward from that baseline.
+    Apply that visual x correction here instead of changing the sensor TFs.
     Baked visual mesh bbox before URDF origin offset:
       x [-0.790, 3.845]
       y [-1.067, 1.067]
       z [0.000, 1.600]
-    Runtime visual bbox after offset:
+    Runtime visual bbox after offsets:
+      x [-0.8400, 3.7950]
       z [-0.3705, 1.2295]
   -->
@@ -25,8 +34,9 @@
   <xacro:property name="vehicle_center_x" value="1.5275"/>
   <xacro:property name="vehicle_center_z" value="0.800"/>
+  <xacro:property name="visual_x_offset" value="-0.0500"/>
   <xacro:property name="visual_z_offset" value="${-wheel_radius}"/>
   <link name="base_link">
     <visual name="ioniq5_visual">
-      <origin xyz="0 0 ${visual_z_offset}" rpy="0 0 0"/>
+      <origin xyz="${visual_x_offset} 0 ${visual_z_offset}" rpy="0 0 0"/>
       <geometry>
         <mesh
@@ -36,5 +46,5 @@
     </visual>
     <collision name="ioniq5_body_box">
-      <origin xyz="${vehicle_center_x} 0 ${vehicle_center_z + visual_z_offset}" rpy="0 0 0"/>
+      <origin xyz="${vehicle_center_x + visual_x_offset} 0 ${vehicle_center_z + visual_z_offset}" rpy="0 0 0"/>
       <geometry>
         <box size="${vehicle_length} ${vehicle_body_width} ${vehicle_height}"/>
